File: hardware/src/HORLJ200319-A/file5EB15525.sch (KiCad schematic (older format))
At the start: 26 parts

Commit message: Insere MockUps digitais e inicia o projeto da PCB.
Parts:
- removed D51, D52, D53, D54, D55, D56, D57, D58, D59, D60, D61, D62, D63, D64, D65: RED, symbol Device:LED_Small_ALT
- removed R25, R26, R27, R28, R29, R30, R31, R32, R33, R34, R35: R_Small, symbol Device:R_Small
